File: USBCtoA2_0.kicad_sch (KiCad schematic)
At the start: 9 parts, among them J1 USB_A, J3 USB_C_Receptacle_USB2.0_16P, U1 USBLC6-2SC6

Commit message: First Trace on PCB
Footprint Assign & PCB Traced
Parts:
- C1: footprint (none) -> Capacitor_SMD:C_1206_3216Metric_Pad1.33x1.80mm_HandSolder
- C2, C3: footprint (none) -> Capacitor_SMD:C_0805_2012Metric_Pad1.18x1.45mm_HandSolder
- F1: footprint (none) -> Fuse:Fuse_1812_4532Metric_Pad1.30x3.40mm_HandSolder
- J1: footprint (none) -> Connector_USB:USB_A_Molex_48037-2200_Horizontal
- J3: footprint (none) -> Connector_USB:USB_C_Receptacle_G-Switch_GT-USB-7010ASV
- R1, R2: footprint (none) -> Resistor_SMD:R_1206_3216Metric_Pad1.30x1.75mm_HandSolder
Connections:
- net +5V: now also J1.1 (VBUS)
- net GND: now also C1.2, C2.2
- net at C1.1, C2.1, F1.1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: now also C3.1, J3.A4 (VBUS), J3.A9 (VBUS), J3.B4 (VBUS), J3.B9 (VBUS), U1.5 (VBUS)
- net D+: now reaches J3.A6 (D+), J3.B6 (D+), U1.1 (I/O1)
- net D-: now reaches J3.A7 (D-), J3.B7 (D-), U1.3 (I/O2)
- net D_out-: now reaches J1.2 (D-), U1.4 (I/O2)
- net D_out+: now reaches J1.3 (D+), U1.6 (I/O1)
- no-connect marks 1 -> 2
Other:
- moved on the sheet: C3
